File: pcb_design/sangaboard_v0.3.kicad_pcb (KiCad board)
At the start: 2 copper layers, 65 x 55 mm, 67 parts, among them J1 USB_Supply, J10 ISP, J11 USB_OTG, J12 X_AXIS, J13 Y_AXIS, J14 Z_AXIS, J2 USB_POWER OUT, J3 END_STOPS, J4 I2C Header, J5 Serial1 Header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

Commit message: Remove diode between usb power in and out
Parts:
- removed ?: , Symbols:OSHW-Logo_5.7x6mm_SilkScreen
- removed ?: , sangaboard_Logo:sangaboard_L5_FS
- removed ?: , sangaboard_Logo:sangaboard_L3_FS
- removed ?: , Symbols:OSHW-Logo_19x20mm_SilkScreen
- removed D2: DW2W31900L, Diodes_SMD:D_SOD-123F
Connections:
- C4 pad 1: Net-(C4-Pad1) -> PWR_OUT
- C5 pad 2: Net-(C4-Pad1) -> PWR_OUT
- D3 pad 2: Net-(C4-Pad1) -> PWR_OUT
- D4 pad 2: Net-(C4-Pad1) -> PWR_OUT
- F1 pad 1: Net-(C4-Pad1) -> PWR_OUT
Routing:
- net Net-(C4-Pad1): track 34.2 -> 0.00 mm
- net PWR_OUT: track 36.7 -> 50.4 mm
Other:
- board text added: "sangaboard v_0.3.1"
- board text removed: "sangaboard v_0.3"
